File: v1/hardware/pcbs/test-boards/BLDC-FOC/power-phase.kicad_sch (KiCad schematic)
At the start: 14 parts, among them Q1 BSC093N15NS5, Q2 BSC093N15NS5

Commit message: larger resistors for high voltages, new prod files
Parts:
- R15, R16: footprint Resistor_SMD:R_0603_1608Metric -> Resistor_SMD:R_0805_2012Metric
Changed lines of the file:
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@@
 			)
 		)
-		(property "Footprint" "Resistor_SMD:R_0603_1608Metric"
+		(property "Footprint" "Resistor_SMD:R_0805_2012Metric"
 			(at 151.13 93.98 0)
 			(effects
@@
 			)
 		)
-		(property "Footprint" "Resistor_SMD:R_0603_1608Metric"
+		(property "Footprint" "Resistor_SMD:R_0805_2012Metric"
 			(at 151.13 99.06 0)
 			(effects
