File: v1/hardware/pcbs/test-boards/BLDC-FOC/power.kicad_sch (KiCad schematic)
At the start: 22 parts, among them P1 WJ500V-5.08-2P-14-00A, Q7 SP015N03BGHTO, Q8 AO3400A_C347475, U2 MX74700T_C22468156, U3 KF88SA-16.0-2P, U4 MX74700T_C22468156, U5 AP63205WU, U6 AZ1117EH-3.3TRG1

Commit message: new FOC driver schematic
Parts:
- C12, C13, C14, C15, C7, C8: symbol Device:C_Small -> symbols:C_Small
- C37, C38, C5, C6: symbol Device:C -> symbols:C
- D4, D5: symbol Device:D_TVS -> symbols:D_TVS
- F1: symbol EasyEDA:R1245.100 -> symbols:R1245.100
- L2: symbol EasyEDA:SL0420-4R7M -> symbols:SL0420-4R7M
- P1: symbol EasyEDA:WJ500V-5.08-2P-14-00A -> symbols:WJ500V-5.08-2P-14-00A
- Q7: symbol EasyEDA:SP015N03BGHTO -> symbols:SP015N03BGHTO
- Q8: symbol EasyEDA:AO3400A_C347475 -> symbols:AO3400A_C347475
- U2, U4: symbol EasyEDA:MX74700T_C22468156 -> symbols:MX74700T_C22468156
- U3: symbol EasyEDA:KF88SA-16.0-2P -> symbols:KF88SA-16.0-2P
- U5: symbol Regulator_Switching:AP63205WU -> symbols:AP63205WU
- U6: symbol EasyEDA:AZ1117EH-3.3TRG1 -> symbols:AZ1117EH-3.3TRG1
Changed lines of the file:
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@@
 	)
 	(symbol
-		(lib_id "EasyEDA:SP015N03BGHTO")
+		(lib_id "symbols:SP015N03BGHTO")
 		(at 129.54 138.43 270)
 		(mirror x)
@@
 	)
 	(symbol
-		(lib_id "Device:C_Small")
+		(lib_id "symbols:C_Small")
 		(at 198.12 50.8 0)
 		(unit 1)
@@
 	)
 	(symbol
-		(lib_id "EasyEDA:MX74700T_C22468156")
+		(lib_id "symbols:MX74700T_C22468156")
 		(at 129.54 81.28 0)
 		(unit 1)
@@
 	)
 	(symbol
-		(lib_id "EasyEDA:KF88SA-16.0-2P")
+		(lib_id "symbols:KF88SA-16.0-2P")
 		(at 133.35 119.38 0)
 		(unit 1)
@@
 	)
 	(symbol
-		(lib_id "EasyEDA:R1245.100")
+		(lib_id "symbols:R1245.100")
 		(at 142.24 135.89 0)
 		(unit 1)
@@
 	)
 	(symbol
-		(lib_id "Device:C_Small")
+		(lib_id "symbols:C_Small")
 		(at 205.74 76.2 0)
 		(unit 1)
@@
 	)
 	(symbol
-		(lib_id "Device:C")
+		(lib_id "symbols:C")
 		(at 107.95 139.7 0)
 		(unit 1)
@@
 	)
 	(symbol
-		(lib_id "Device:C_Small")
+		(lib_id "symbols:C_Small")
 		(at 273.05 48.26 0)
 		(unit 1)
@@
 	)
 	(symbol
-		(lib_id "Device:C")
+		(lib_id "symbols:C")
 		(at 129.54 67.31 270)
 		(unit 1)
@@
 	)
 	(symbol
-		(lib_id "Device:D_TVS")
+		(lib_id "symbols:D_TVS")
 		(at 92.71 53.34 90)
 		(unit 1)
@@
 	)
 	(symbol
-		(lib_id "Device:C_Small")
+		(lib_id "symbols:C_Small")
 		(at 240.03 48.26 0)
 		(unit 1)
@@
 	)
 	(symbol
-		(lib_id "Device:C")
+		(lib_id "symbols:C")
 		(at 107.95 53.34 0)
 		(unit 1)
@@
 	)
 	(symbol
-		(lib_id "power:PWR_FLAG")
+		(lib_id "symbols:PWR_FLAG")
 		(at 109.22 120.65 90)
 		(unit 1)
@@
 	)
 	(symbol
-		(lib_id "Device:D_TVS")
+		(lib_id "symbols:D_TVS")
 		(at 92.71 139.7 90)
 		(unit 1)
@@
 	)
 	(symbol
-		(lib_id "Device:C_Small")
+		(lib_id "symbols:C_Small")
 		(at 259.08 48.26 0)
 		(unit 1)
@@
 	)
 	(symbol
-		(lib_id "power:PWR_FLAG")
+		(lib_id "symbols:PWR_FLAG")
 		(at 266.7 45.72 0)
 		(unit 1)
@@
 	)
 	(symbol
-		(lib_id "power:PWR_FLAG")
+		(lib_id "symbols:PWR_FLAG")
 		(at 111.76 33.02 90)
 		(unit 1)
@@
 	)
 	(symbol
-		(lib_id "Regulator_Switching:AP63205WU")
+		(lib_id "symbols:AP63205WU")
 		(at 222.25 50.8 0)
 		(unit 1)
@@
 	)
 	(symbol
-		(lib_id "EasyEDA:SL0420-4R7M")
+		(lib_id "symbols:SL0420-4R7M")
 		(at 250.19 45.72 0)
 		(unit 1)
@@
 	)
 	(symbol
-		(lib_id "EasyEDA:AO3400A_C347475")
+		(lib_id "symbols:AO3400A_C347475")
 		(at 129.54 49.53 270)
 		(mirror x)
@@
 	)
 	(symbol
-		(lib_id "EasyEDA:WJ500V-5.08-2P-14-00A")
+		(lib_id "symbols:WJ500V-5.08-2P-14-00A")
 		(at 133.35 34.29 270)
 		(unit 1)
@@
 	)
 	(symbol
-		(lib_id "Device:C_Small")
+		(lib_id "symbols:C_Small")
 		(at 236.22 76.2 0)
 		(unit 1)
@@
 	)
 	(symbol
-		(lib_id "EasyEDA:AZ1117EH-3.3TRG1")
+		(lib_id "symbols:AZ1117EH-3.3TRG1")
 		(at 222.25 78.74 0)
 		(unit 1)
@@
 	)
 	(symbol
-		(lib_id "power:PWR_FLAG")
+		(lib_id "symbols:PWR_FLAG")
 		(at 148.59 139.7 180)
 		(unit 1)
@@
 	)
 	(symbol
-		(lib_id "Device:C")
+		(lib_id "symbols:C")
 		(at 129.54 153.67 270)
 		(unit 1)
@@
 	)
 	(symbol
-		(lib_id "EasyEDA:MX74700T_C22468156")
+		(lib_id "symbols:MX74700T_C22468156")
 		(at 129.54 167.64 0)
 		(unit 1)
