File: v1/hardware/pcbs/test-boards/STM32G491CET6/STM32G491CET6.kicad_pcb (KiCad board)
At the start: 2 copper layers, 43 x 38 mm, 45 parts, among them J1 Conn_02x10_Odd_Even, J2 Conn_02x10_Odd_Even, J3 Conn_01x04, U1 STM32G491CETx, Y1 Crystal_GND24, Y2 Crystal

Commit message: new FOC driver schematic
Parts:
- BOOT1, RESET1: footprint EasyEDA:SW-SMD_L3.1-W3.1-P2.20-LS4.0 -> footprints:SW-SMD_L3.1-W3.1-P2.20-LS4.0
- C1, C10, C11, C12, C13, C14, C2, C3, C4, C5, C6, C7, C8, C9: footprint Capacitor_SMD:C_0603_1608Metric -> footprints:C_0603_1608Metric
- D1, D2: footprint Diode_SMD:D_0603_1608Metric -> footprints:D_0603_1608Metric
- D3: footprint Diode_SMD:D_SOD-123F -> footprints:D_SOD-123F
- D4, D5: footprint Diode_SMD:D_SOD-323 -> footprints:D_SOD-323
- FB1: footprint Inductor_SMD:L_0603_1608Metric -> footprints:L_0603_1608Metric
- H1, H2, H3: footprint MountingHole:MountingHole_3.2mm_M3_Pad_Via -> footprints:MountingHole_3.2mm_M3_Pad_Via
- J1, J2: footprint Connector_PinHeader_2.54mm:PinHeader_2x10_P2.54mm_Vertical -> footprints:PinHeader_2x10_P2.54mm_Vertical
- J3: footprint Connector_PinHeader_2.54mm:PinHeader_1x04_P2.54mm_Vertical -> footprints:PinHeader_1x04_P2.54mm_Vertical
- LDO1: footprint Package_TO_SOT_SMD:SOT-23-5 -> footprints:SOT-23-5
- LED1, LED2: footprint LED_SMD:LED_0603_1608Metric -> footprints:LED_0603_1608Metric
- R1, R2, R3, R4, R5, R6, R7, R8, R9: footprint Resistor_SMD:R_0603_1608Metric -> footprints:R_0603_1608Metric
- U1: footprint Package_QFP:LQFP-48_7x7mm_P0.5mm -> footprints:LQFP-48_7x7mm_P0.5mm
- USB1: footprint EasyEDA:USB-C-SMD_TYPE-C-6PIN-2MD-073 -> footprints:USB-C-SMD_TYPE-C-6PIN-2MD-073
- USBPWR1: footprint Connector_PinHeader_2.54mm:PinHeader_1x02_P2.54mm_Vertical -> footprints:PinHeader_1x02_P2.54mm_Vertical
- Y1: footprint Crystal:Crystal_SMD_3225-4Pin_3.2x2.5mm -> footprints:Crystal_SMD_3225-4Pin_3.2x2.5mm
- Y2: footprint Crystal:Crystal_SMD_3215-2Pin_3.2x1.5mm -> footprints:Crystal_SMD_3215-2Pin_3.2x1.5mm
Changed lines of the file:
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@@
 	(net 79 "unconnected-(H3-Pad1)_7")
 	(net 80 "unconnected-(H3-Pad1)_8")
-	(footprint "Capacitor_SMD:C_0603_1608Metric"
+	(footprint "footprints:C_0603_1608Metric"
 		(layer "F.Cu")
 		(at -5.15 -2.675 90)
@@
 		)
 	)
-	(footprint "Resistor_SMD:R_0603_1608Metric"
+	(footprint "footprints:R_0603_1608Metric"
 		(layer "F.Cu")
 		(at -6.8 9.2)
@@
 		)
 	)
-	(footprint "Capacitor_SMD:C_0603_1608Metric"
+	(footprint "footprints:C_0603_1608Metric"
 		(layer "F.Cu")
 		(at 15.9 14.8 180)
@@
 		)
 	)
-	(footprint "Inductor_SMD:L_0603_1608Metric"
+	(footprint "footprints:L_0603_1608Metric"
 		(layer "F.Cu")
 		(at 8.35 7.9)
@@
 		)
 	)
-	(footprint "Capacitor_SMD:C_0603_1608Metric"
+	(footprint "footprints:C_0603_1608Metric"
 		(layer "F.Cu")
 		(at -6.25 1.475 -90)
@@
 		)
 	)
-	(footprint "Crystal:Crystal_SMD_3225-4Pin_3.2x2.5mm"
+	(footprint "footprints:Crystal_SMD_3225-4Pin_3.2x2.5mm"
 		(layer "F.Cu")
 		(at -3.7 1.475 -90)
@@
 		)
 	)
-	(footprint "MountingHole:MountingHole_3.2mm_M3_Pad_Via"
+	(footprint "footprints:MountingHole_3.2mm_M3_Pad_Via"
 		(layer "F.Cu")
 		(at 17.5 -15)
@@
 		(embedded_fonts no)
 	)
-	(footprint "Resistor_SMD:R_0603_1608Metric"
+	(footprint "footprints:R_0603_1608Metric"
 		(layer "F.Cu")
 		(at -9.4 -9.6 45)
@@
 		)
 	)
-	(footprint "Capacitor_SMD:C_0603_1608Metric"
+	(footprint "footprints:C_0603_1608Metric"
 		(layer "F.Cu")
 		(at 5.25 6.3)
@@
 		)
 	)
-	(footprint "Package_QFP:LQFP-48_7x7mm_P0.5mm"
+	(footprint "footprints:LQFP-48_7x7mm_P0.5mm"
 		(layer "F.Cu")
 		(at 4.5 0)
@@
 		)
 	)
-	(footprint "Connector_PinHeader_2.54mm:PinHeader_1x02_P2.54mm_Vertical"
+	(footprint "footprints:PinHeader_1x02_P2.54mm_Vertical"
 		(layer "F.Cu")
 		(at 19.5 7 -90)
@@
 		)
 	)
-	(footprint "Resistor_SMD:R_0603_1608Metric"
+	(footprint "footprints:R_0603_1608Metric"
 		(layer "F.Cu")
 		(at 13.5 9.2 -90)
@@
 		)
 	)
-	(footprint "Crystal:Crystal_SMD_3215-2Pin_3.2x1.5mm"
+	(footprint "footprints:Crystal_SMD_3215-2Pin_3.2x1.5mm"
 		(layer "F.Cu")
 		(at -3.15 -3.15 90)
@@
 		)
 	)
-	(footprint "LED_SMD:LED_0603_1608Metric"
+	(footprint "footprints:LED_0603_1608Metric"
 		(layer "F.Cu")
 		(at -10 9.2)
@@
 		)
 	)
-	(footprint "EasyEDA:USB-C-SMD_TYPE-C-6PIN-2MD-073"
+	(footprint "footprints:USB-C-SMD_TYPE-C-6PIN-2MD-073"
 		(layer "F.Cu")
 		(at 16.4175 0 90)
@@
 		)
 	)
-	(footprint "Resistor_SMD:R_0603_1608Metric"
+	(footprint "footprints:R_0603_1608Metric"
 		(layer "F.Cu")
 		(at 17.2 -7.2 -90)
@@
 		)
 	)
-	(footprint "Diode_SMD:D_0603_1608Metric"
+	(footprint "footprints:D_0603_1608Metric"
 		(layer "F.Cu")
 		(at -3.5 -7.6 180)
@@
 		)
 	)
-	(footprint "Resistor_SMD:R_0603_1608Metric"
+	(footprint "footprints:R_0603_1608Metric"
 		(layer "F.Cu")
 		(at 20.4 -7.2 -90)
@@
 		)
 	)
-	(footprint "EasyEDA:SW-SMD_L3.1-W3.1-P2.20-LS4.0"
+	(footprint "footprints:SW-SMD_L3.1-W3.1-P2.20-LS4.0"
 		(layer "F.Cu")
 		(at -8.9 4 90)
@@
 		)
 	)
-	(footprint "Capacitor_SMD:C_0603_1608Metric"
+	(footprint "footprints:C_0603_1608Metric"
 		(layer "F.Cu")
 		(at -3.45 -6 180)
@@
 		)
 	)
-	(footprint "Diode_SMD:D_SOD-323"
+	(footprint "footprints:D_SOD-323"
 		(layer "F.Cu")
 		(at 12.1 1.8 -90)
@@
 		)
 	)
-	(footprint "Package_TO_SOT_SMD:SOT-23-5"
+	(footprint "footprints:SOT-23-5"
 		(layer "F.Cu")
 		(at 19.3 13.4 -90)
@@
 		)
 	)
-	(footprint "Capacitor_SMD:C_0603_1608Metric"
+	(footprint "footprints:C_0603_1608Metric"
 		(layer "F.Cu")
 		(at -3.625 4.425 180)
@@
 		)
 	)
-	(footprint "Capacitor_SMD:C_0603_1608Metric"
+	(footprint "footprints:C_0603_1608Metric"
 		(layer "F.Cu")
 		(at 14 -7.2 90)
@@
 		)
 	)
-	(footprint "Resistor_SMD:R_0603_1608Metric"
+	(footprint "footprints:R_0603_1608Metric"
 		(layer "F.Cu")
 		(at 2.7 -7.4 90)
@@
 		)
 	)
-	(footprint "Resistor_SMD:R_0603_1608Metric"
+	(footprint "footprints:R_0603_1608Metric"
 		(layer "F.Cu")
 		(at -3.5 -9.2 180)
@@
 		)
 	)
-	(footprint "LED_SMD:LED_0603_1608Metric"
+	(footprint "footprints:LED_0603_1608Metric"
 		(layer "F.Cu")
 		(at 12.943153 5.843153 -45)
@@
 		)
 	)
-	(footprint "Diode_SMD:D_SOD-123F"
+	(footprint "footprints:D_SOD-123F"
 		(layer "F.Cu")
 		(at 18.9 10)
@@
 		)
 	)
-	(footprint "MountingHole:MountingHole_3.2mm_M3_Pad_Via"
+	(footprint "footprints:MountingHole_3.2mm_M3_Pad_Via"
 		(layer "F.Cu")
 		(at -17.5 15)
@@
 		(embedded_fonts no)
 	)
-	(footprint "Capacitor_SMD:C_0603_1608Metric"
+	(footprint "footprints:C_0603_1608Metric"
 		(layer "F.Cu")
 		(at 9.1 -4.75 -90)
@@
 		)
 	)
-	(footprint "Capacitor_SMD:C_0603_1608Metric"
+	(footprint "footprints:C_0603_1608Metric"
 		(layer "F.Cu")
 		(at 0.1 8 90)
@@
 		)
 	)
-	(footprint "EasyEDA:SW-SMD_L3.1-W3.1-P2.20-LS4.0"
+	(footprint "footprints:SW-SMD_L3.1-W3.1-P2.20-LS4.0"
 		(layer "F.Cu")
 		(at -8.9 -4 90)
@@
 		)
 	)
-	(footprint "MountingHole:MountingHole_3.2mm_M3_Pad_Via"
+	(footprint "footprints:MountingHole_3.2mm_M3_Pad_Via"
 		(layer "F.Cu")
 		(at -17.5 -15)
@@
 		(embedded_fonts no)
 	)
-	(footprint "Capacitor_SMD:C_0603_1608Metric"
+	(footprint "footprints:C_0603_1608Metric"
 		(layer "F.Cu")
 		(at 15.9 12.2 180)
@@
 		)
 	)
-	(footprint "Capacitor_SMD:C_0603_1608Metric"
+	(footprint "footprints:C_0603_1608Metric"
 		(layer "F.Cu")
 		(at 8.5 5.35 90)
@@
 		)
 	)
-	(footprint "Resistor_SMD:R_0603_1608Metric"
+	(footprint "footprints:R_0603_1608Metric"
 		(layer "F.Cu")
 		(at 18.8 -7.2 90)
@@
 		)
 	)
-	(footprint "Capacitor_SMD:C_0603_1608Metric"
+	(footprint "footprints:C_0603_1608Metric"
 		(layer "F.Cu")
 		(at -1.1 -5.35 -90)
@@
 		)
 	)
-	(footprint "Diode_SMD:D_0603_1608Metric"
+	(footprint "footprints:D_0603_1608Metric"
 		(layer "F.Cu")
 		(at 0.3 -9.4 180)
@@
 		)
 	)
-	(footprint "Capacitor_SMD:C_0603_1608Metric"
+	(footprint "footprints:C_0603_1608Metric"
 		(layer "F.Cu")
 		(at 5.25 7.9)
@@
 		)
 	)
-	(footprint "Capacitor_SMD:C_0603_1608Metric"
+	(footprint "footprints:C_0603_1608Metric"
 		(layer "F.Cu")
 		(at 0.5 -5.35 -90)
@@
 		)
 	)
-	(footprint "Diode_SMD:D_SOD-323"
+	(footprint "footprints:D_SOD-323"
 		(layer "F.Cu")
 		(at 12.1 -1.8 90)
@@
 		)
 	)
-	(footprint "Connector_PinHeader_2.54mm:PinHeader_1x04_P2.54mm_Vertical"
+	(footprint "footprints:PinHeader_1x04_P2.54mm_Vertical"
 		(layer "F.Cu")
 		(at -12.9 -3.81)
@@
 		)
 	)
-	(footprint "Resistor_SMD:R_0603_1608Metric"
+	(footprint "footprints:R_0603_1608Metric"
 		(layer "F.Cu")
 		(at 15.6 -7.2 90)
@@
 		)
 	)
-	(footprint "Connector_PinHeader_2.54mm:PinHeader_2x10_P2.54mm_Vertical"
+	(footprint "footprints:PinHeader_2x10_P2.54mm_Vertical"
 		(layer "B.Cu")
 		(at 11.43 -13.97 90)
@@
 		)
 	)
-	(footprint "Connector_PinHeader_2.54mm:PinHeader_2x10_P2.54mm_Vertical"
+	(footprint "footprints:PinHeader_2x10_P2.54mm_Vertical"
 		(layer "B.Cu")
 		(at 11.43 16.51 90)
