File: v1/hardware/pcbs/FOC-driver/FOC-driver.kicad_pcb (KiCad board)
At the start: 4 copper layers, 100 x 100 mm, 223 parts, among them J1 HB9500M-9.5-2P, J10 S4B-XH-A, J11 S10B-XH-A, J12 S8B-XH-A, J13 S5B-XH-A, J14 S2B-XH-A, J15 S5B-XH-A, J16 S2B-XH-A, J2 HB9500-3, J3 B2B-XH-A, J4 B2B-XH-A, J5 B2B-XH-A, J6 B2B-XH-A, J7 S2B-XH-A, J8 S5B-XH-A, J9 S4B-XH-A, Q1 BSC093N15NS5, Q10 40N05, Q11 40N05, Q2 BSC093N15NS5, Q3 BSC093N15NS5, Q4 BSC093N15NS5, Q5 BSC093N15NS5, Q6 BSC093N15NS5, Q7 SP015N03BGHTO, Q8 40N05, Q9 40N05, SW1 TS-1088-AR02016, SW2 MSK22D18G2 125, Y1 C19674287, Y2 C48615

Commit message: new FOC driver done
Parts:
- removed C31: 100nF 50V, Capacitor_SMD:C_0402_1005Metric
- removed C32: 1uF 16V, Capacitor_SMD:C_0402_1005Metric
- removed C4: 820uF 100V (C443165), Capacitor_THT:C_Radial_D18.0mm_H35.5mm_P7.50mm
- removed R4: 4.7K, Resistor_SMD:R_0402_1005Metric
- removed R5: 1K, Resistor_SMD:R_0402_1005Metric
- removed TH1, TH2, TH3, TH4, TH5, TH6: NCP15XH103F03RC, Resistor_SMD:R_0402_1005Metric
- removed TP17: TestPoint, Connector_PinSocket_2.54mm:PinSocket_1x01_P2.54mm_Vertical
- added C70: 100nF 50V, Capacitor_SMD:C_0402_1005Metric, F.Cu at (0.80, 0.00)
- added J17: B2B-XH-A, Connector_JST:JST_XH_B2B-XH-A_1x02_P2.50mm_Vertical, F.Cu at (23.0, -0.25)
- added J18: B2B-XH-A, Connector_JST:JST_XH_B2B-XH-A_1x02_P2.50mm_Vertical, F.Cu at (23.0, -7.00)
- added J19: B2B-XH-A, Connector_JST:JST_XH_B2B-XH-A_1x02_P2.50mm_Vertical, F.Cu at (23.0, 13.2)
- added J20: B2B-XH-A, Connector_JST:JST_XH_B2B-XH-A_1x02_P2.50mm_Vertical, F.Cu at (23.0, 6.50)
- added J21: B2B-XH-A, Connector_JST:JST_XH_B2B-XH-A_1x02_P2.50mm_Vertical, F.Cu at (23.0, 26.8)
- added J22: B2B-XH-A, Connector_JST:JST_XH_B2B-XH-A_1x02_P2.50mm_Vertical, F.Cu at (23.0, 20.0)
- added R68: 10K, Resistor_SMD:R_0402_1005Metric, F.Cu at (-15.8, -26.2)
- added R69: 10K, Resistor_SMD:R_0402_1005Metric, F.Cu at (27.6, 20.8)
- added R70: 10K, Resistor_SMD:R_0402_1005Metric, F.Cu at (27.6, -14.2)
- added R71: 10K, Resistor_SMD:R_0402_1005Metric, F.Cu at (27.6, 27.8)
- added R72: 10K, Resistor_SMD:R_0402_1005Metric, F.Cu at (27.6, 13.8)
- added R73: 10K, Resistor_SMD:R_0402_1005Metric, F.Cu at (27.6, 34.8)
- added R74: 10K, Resistor_SMD:R_0402_1005Metric, F.Cu at (16.8, 34.8)
- added R75: 100, Resistor_SMD:R_0402_1005Metric, F.Cu at (35.9, 34.0)
- added R76: 100, Resistor_SMD:R_0402_1005Metric, F.Cu at (25.2, 34.0)
- added TP8: PinHeader 1x1, Connector_PinHeader_2.54mm:PinHeader_1x01_P2.54mm_Vertical, F.Cu at (-23.6, 9.40)
- TP1, TP2, TP3, TP4, TP5, TP6, TP7: value TestPoint -> PinHeader 1x1; footprint Connector_PinSocket_2.54mm:PinSocket_1x01_P2.54mm_Vertical -> Connector_PinHeader_2.54mm:PinHeader_1x01_P2.54mm_Vertical
- moved DIFF_RECV6 246.5 mm to (31.8, 34.0)
- moved C52 244.0 mm to (35.0, 31.0), turned to 180 degrees
- moved DIFF_RECV7 241.2 mm to (21.0, 34.0)
- moved C71 240.5 mm to (37.8, -47.0), turned to -90 degrees
- moved C69 240.4 mm to (40.0, -41.8), turned to 180 degrees
- moved C68 240.2 mm to (40.0, -43.2), turned to 180 degrees
- moved C67 240.0 mm to (40.0, -44.8), turned to 180 degrees
- moved C66 239.8 mm to (40.0, -46.2), turned to 180 degrees
- moved C16 239.6 mm to (40.0, -47.8), turned to 180 degrees
- moved C64 235.6 mm to (24.2, 31.0), turned to 180 degrees
- moved C41 229.8 mm to (21.8, -42.2), turned to -90 degrees
- moved C42 222.7 mm to (13.8, -39.0), turned to -90 degrees
- moved C40 222.7 mm to (35.0, -11.0), turned to 180 degrees
- moved C44 222.3 mm to (17.8, -29.2), turned to -90 degrees
- moved C43 221.3 mm to (14.0, -34.4), turned to -90 degrees
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Connections:
- net Net-(C41-Pad2) renamed /CANTERM_MID
- C10 pad 1: /VS2 -> /V_POWER
- C11 pad 1: /VS3 -> /U_POWER
- C9 pad 1: /VS1 -> /W_POWER
- DIFF_RECV1 pad 4: unconnected-(DIFF_RECV1-DI-Pad4) -> Net-(DIFF_RECV1-DI)
- DIFF_RECV2 pad 4: unconnected-(DIFF_RECV2-DI-Pad4) -> Net-(DIFF_RECV2-DI)
- DIFF_RECV3 pad 4: unconnected-(DIFF_RECV3-DI-Pad4) -> Net-(DIFF_RECV3-DI)
- DIFF_RECV4 pad 4: unconnected-(DIFF_RECV4-DI-Pad4) -> Net-(DIFF_RECV4-DI)
- DIFF_RECV5 pad 4: unconnected-(DIFF_RECV5-DI-Pad4) -> Net-(DIFF_RECV5-DI)
- DIFF_RECV6 pad 4: unconnected-(DIFF_RECV6-DI-Pad4) -> Net-(DIFF_RECV6-DI)
- DIFF_RECV7 pad 4: unconnected-(DIFF_RECV7-DI-Pad4) -> Net-(DIFF_RECV7-DI)
- GDRV1 pad 1: /U_LOW_PWM -> /W_LOW_PWM
- GDRV1 pad 11: /U_LOW_GATE -> /W_LOW_GATE
- GDRV1 pad 12: /VS3 -> /U_POWER
- GDRV1 pad 13: /W_HIGH_GATE -> /U_HIGH_GATE
- GDRV1 pad 15: /VS2 -> /V_POWER
- GDRV1 pad 18: /VS1 -> /W_POWER
- GDRV1 pad 19: /U_HIGH_GATE -> /W_HIGH_GATE
- GDRV1 pad 22: /U_HIGH_PWM -> /W_HIGH_PWM
- GDRV1 pad 24: /W_HIGH_PWM -> /U_HIGH_PWM
- GDRV1 pad 3: /W_LOW_PWM -> /U_LOW_PWM
- GDRV1 pad 9: /W_LOW_GATE -> /U_LOW_GATE
- J13 pad 2: /RS422.TX+ -> /RS422.RX-
- J13 pad 3: /RS422.TX- -> /RS422.RX+
- J13 pad 4: /RS422.RX+ -> /RS422.TX-
- J13 pad 5: /RS422.RX- -> /RS422.TX+
- J15 pad 2: /NRST -> /DEBUG.SWDIO
- J15 pad 4: /DEBUG.SWDIO -> /DEBUG.SWO
- J15 pad 5: /DEBUG.SWO -> /NRST
- J8 pad 2: /FDCAN.CAN+ -> /FDCAN.CAN-
- J8 pad 3: /FDCAN.CAN- -> /FDCAN.CAN+
- J8 pad 4: /FDCAN.CAN- -> /FDCAN.CAN+
- J8 pad 5: /FDCAN.CAN+ -> /FDCAN.CAN-
- MCU1 pad 10: /V_LOW_TEMP -> /W_LOW_TEMP
- MCU1 pad 11: /W_HIGH_TEMP -> /V_HIGH_TEMP
- MCU1 pad 12: /12V_SENSE -> /V_LOW_TEMP
- MCU1 pad 13: /5V_SENSE -> /U_HIGH_TEMP
- MCU1 pad 14: /U_HIGH_TEMP -> /U_LOW_TEMP
- MCU1 pad 17: /U_LOW_TEMP -> /12V_SENSE
- MCU1 pad 2: /U_LOW_PWM -> /W_LOW_PWM
- MCU1 pad 20: /VMOT_SENSE -> /MOTOR_TEMP
- MCU1 pad 22: /W_LOW_TEMP -> /VMOT_SENSE
- MCU1 pad 25: /W_LOW_PWM -> /U_LOW_PWM
- MCU1 pad 26: /FAN1.EN -> /ENC.SCS
- MCU1 pad 30: /DIP.CONF0 -> /FAN4.EN
- MCU1 pad 33: /DIP.CONF1 -> /FAN3.EN
- MCU1 pad 34: /DIP.CONF2 -> /FAN2.EN
- MCU1 pad 37: /ENC.SCS -> /FAN1.EN
- MCU1 pad 39: /FAN2.PWM -> /FAN3.PWM
- MCU1 pad 40: /FAN3.PWM -> /FAN2.PWM
- MCU1 pad 41: /FAN4.PWM -> /FAN1.PWM
- MCU1 pad 42: /U_HIGH_PWM -> /W_HIGH_PWM
- MCU1 pad 44: /W_HIGH_PWM -> /U_HIGH_PWM
- MCU1 pad 51: /FAN1.PWM -> /FAN4.PWM
- MCU1 pad 52: /FAN4.EN -> /DIP.CONF2
- MCU1 pad 53: /FAN3.EN -> /DIP.CONF1
- MCU1 pad 54: /FAN2.EN -> /DIP.CONF0
- MCU1 pad 62: /ENDSTOP2 -> /ENDSTOP1
- MCU1 pad 8: /ENDSTOP1 -> /ENDSTOP2
- MCU1 pad 9: /V_HIGH_TEMP -> /W_HIGH_TEMP
- R35 pad 2: Net-(R35-Pad2) -> /CANTERM+
- R36 pad 2: Net-(R36-Pad2) -> /CANTERM-
- SW2 pad 1: unconnected-(SW2-Pad1) -> GND
- SW2 pad 2: /FDCAN.CAN+ -> /CANTERM+
- SW2 pad 3: Net-(R36-Pad2) -> /FDCAN.CAN+
- SW2 pad 4: unconnected-(SW2-Pad4) -> GND
- SW2 pad 5: /FDCAN.CAN- -> /CANTERM-
- SW2 pad 6: Net-(R35-Pad2) -> /FDCAN.CAN-
- TP5 pad 1: +12V -> VMOT
- TP6 pad 1: VMOT -> +12V
- TP7 pad 1: GND -> +5V
Routing:
- net +3.3V: track 16.8 -> 407.3 mm, vias 0 -> 12
- net +12V: track 59.9 -> 306.6 mm, vias 0 -> 8
- net +5V: track 15.8 -> 255.3 mm, vias 0 -> 3
- net GND: track 214.5 -> 412.4 mm, vias 103 -> 211
- net /NRST: track 0.00 -> 91.2 mm
- net /DEBUG.SWCLK: track 0.00 -> 84.5 mm
- net /DEBUG.SWO: track 0.00 -> 84.3 mm
- net /DEBUG.SWDIO: track 0.00 -> 83.7 mm
- net /ENDSTOP1: track 0.00 -> 81.0 mm, vias 0 -> 6
- net /ENC.A: track 0.00 -> 71.9 mm, vias 0 -> 6
- net /ENDSTOP2: track 0.00 -> 59.1 mm, vias 0 -> 2
- net /W_I_SENSE: track 4.91 -> 61.9 mm, vias 0 -> 6
- net /ENC.B: track 0.00 -> 55.5 mm, vias 0 -> 2
- net /W_HIGH_TEMP: track 0.00 -> 52.7 mm
- net /ENC.Z: track 0.00 -> 51.0 mm, vias 0 -> 2
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- added copper zone on In1.Cu, net GND
- added copper zone on In2.Cu, net VMOT
Other:
- board text added: "12V"
- board text added: "3.3V"
- board text added: "5V"
- board text added: "B0 C0 C1 C2"
- board text added: "GND"
- board text added: "ON=HIGH"
- board text added: "RESET"
- board text added: "U_HIGH TH"
- board text added: "U_LOW TH"
- board text added: "U_PWR"
- board text added: "VMOT"
- board text added: "V_HIGH TH"
- board text added: "V_LOW TH"
- board text added: "V_PWR"
- board text added: "W_HIGH TH"
- board text added: "W_LOW TH"
- board text added: "W_PWR"

Commit message: added text to new FOC driver
Other:
- board text added: "Maximum ratings: VCC <= 80V, RMS current <= 50A"
- board text added: "foosball bot FOC driver V2 by LJY"
Changed lines of the file:
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@@
+		)
+	)
+	(gr_text "foosball bot\nFOC driver V2 by LJY"
+		(at 12.8 14 0)
+		(layer "B.SilkS")
+		(effects
+			(font
+				(size 2 2)
+				(thickness 0.25)
+			)
+			(justify left bottom mirror)
+		)
+	)
+	(gr_text "Maximum ratings: VCC <= 80V, RMS current <= 50A"
+		(at 12.6 16.35 0)
+		(layer "B.SilkS")
+		(effects
+			(font
+				(size 1.25 1.25)
+				(thickness 0.15625)
+			)
+			(justify left bottom mirror)
 		)
 	)
