File: v1/hardware/pcbs/endstop-switch/endstop-switch.kicad_pcb (KiCad board)
At the start: 2 copper layers, 75 x 40 mm, 8 parts, among them J1 S4B-XH-A, SW1 D2F-L-A

Commit message: misc
Parts:
- moved C1 23.0 mm to (28.2, -5.50)
- moved C2 23.0 mm to (27.5, 2.50)
- moved DIFF_DRV1 23.0 mm to (26.0, -6.25)
- moved J1 23.0 mm to (32.5, 3.75)
- moved R1 23.0 mm to (26.0, -3.75)
- moved SW1 23.0 mm to (29.5, -11.0)
Other:
- board size 75 x 40 mm -> 52 x 40 mm
